Commit message: Match the CallM MuJoCo model: arm mount and base inertia
The mount link is now the UR5e base_link pose from the CallM MuJoCo
model: 15 mm along base +y (tape-measured) and turned +90 deg. The old
-90 deg fit the UR controller base frame, which is base_link turned by
pi, so an arm placed on mount pointed backwards. The RSDF Base surface
gets the same pose. The base mass and inertia come from the MuJoCo
model (120.95 kg, CoM 0.035 m above the floor).

File: urdf/triorb.urdf (robot description, URDF)
Before this commit: robot triorb, 6 links, 5 joints
Links:
- link base: mass 0.1 -> 120.95
Joints:
- joint base_to_mount: origin xyz=0 0 0.30 rpy=0 0 -1.57079632679 -> xyz=0 0.015 0.30 rpy=0 0 1.57079632679
